Commit message: collada format for meshes in rvizweb

File: reconcycle_description/urdf/table_module.xacro (robot description, xacro)
@@ -19,5 +19,5 @@
             <origin rpy="${pi/2} 0 0" xyz=" 0 0 0 "/>
             <geometry>
-                <mesh filename="package://reconcycle_description/meshes/table.obj" scale="0.001 0.001 0.001"/>
+                <mesh filename="package://reconcycle_description/meshes/table.dae" scale="0.001 0.001 0.001"/>
             </geometry>
         </visual>
@@ -25,5 +25,5 @@
             <origin rpy="${pi/2} 0 0" xyz="0.0 0.0 0"/>
             <geometry>
-                <mesh filename="package://reconcycle_description/meshes/table.obj" scale="0.001 0.001 0.001"/>
+                <mesh filename="package://reconcycle_description/meshes/table.dae" scale="0.001 0.001 0.001"/>
             </geometry>
         </collision>
@@ -39,5 +39,5 @@
             <origin rpy="${pi/2} 0 ${pi/2}" xyz=" 0 0 0 "/>
             <geometry>
-                <mesh filename="package://reconcycle_description/meshes/pnp.obj" scale="0.001 0.001 0.001"/>
+                <mesh filename="package://reconcycle_description/meshes/pnp.dae" scale="0.001 0.001 0.001"/>
             </geometry>
         </visual>
@@ -45,5 +45,5 @@
             <origin rpy="${pi/2} 0 ${pi/2}" xyz=" 0 0 0 "/>
             <geometry>
-                <mesh filename="package://reconcycle_description/meshes/pnp.obj" scale="0.001 0.001 0.001"/>
+                <mesh filename="package://reconcycle_description/meshes/pnp.dae" scale="0.001 0.001 0.001"/>
             </geometry>
         </collision>
@@ -58,5 +58,5 @@
             <origin rpy="${pi/2} 0 ${pi/2}" xyz=" 0 0 0 "/>
             <geometry>
-                <mesh filename="package://reconcycle_description/meshes/pnp.obj" scale="0.001 0.001 0.001"/>
+                <mesh filename="package://reconcycle_description/meshes/pnp.dae" scale="0.001 0.001 0.001"/>
             </geometry>
         </visual>
@@ -64,5 +64,5 @@
             <origin rpy="${pi/2} 0 ${pi/2}" xyz=" 0 0 0 "/>
             <geometry>
-                <mesh filename="package://reconcycle_description/meshes/pnp.obj" scale="0.001 0.001 0.001"/>
+                <mesh filename="package://reconcycle_description/meshes/pnp.dae" scale="0.001 0.001 0.001"/>
             </geometry>
         </collision>
@@ -77,5 +77,5 @@
             <origin rpy="${pi/2} 0 ${pi/2}" xyz=" 0 0 0 "/>
             <geometry>
-                <mesh filename="package://reconcycle_description/meshes/pnp.obj" scale="0.001 0.001 0.001"/>
+                <mesh filename="package://reconcycle_description/meshes/pnp.dae" scale="0.001 0.001 0.001"/>
             </geometry>
         </visual>
@@ -83,5 +83,5 @@
             <origin rpy="${pi/2} 0 ${pi/2}" xyz=" 0 0 0 "/>
             <geometry>
-                <mesh filename="package://reconcycle_description/meshes/pnp.obj" scale="0.001 0.001 0.001"/>
+                <mesh filename="package://reconcycle_description/meshes/pnp.dae" scale="0.001 0.001 0.001"/>
             </geometry>
         </collision>
@@ -96,5 +96,5 @@
             <origin rpy="${pi/2} 0 ${pi/2}" xyz=" 0 0 0 "/>
             <geometry>
-                <mesh filename="package://reconcycle_description/meshes/pnp.obj" scale="0.001 0.001 0.001"/>
+                <mesh filename="package://reconcycle_description/meshes/pnp.dae" scale="0.001 0.001 0.001"/>
             </geometry>
         </visual>
@@ -102,5 +102,5 @@
             <origin rpy="${pi/2} 0 ${pi/2}" xyz=" 0 0 0 "/>
             <geometry>
-                <mesh filename="package://reconcycle_description/meshes/pnp.obj" scale="0.001 0.001 0.001"/>
+                <mesh filename="package://reconcycle_description/meshes/pnp.dae" scale="0.001 0.001 0.001"/>
             </geometry>
         </collision>
