Commit message: xacro rotation try

File: reconcycle_description/urdf/actual_layout.xacro (robot description, xacro)
@@ -14,10 +14,10 @@
     <xacro:arg name="table_5_name" default="table_rob_2"/>
     <!-- <xacro:arg name="table_6_name" default="table_parts"/> -->
-    <xacro:table_module table_id="$(arg table_0_name)" connected_to="world" xyz="0 0 ${table_height}"/>
-    <xacro:table_module table_id="$(arg table_1_name)" connected_to="$(arg table_0_name)" xyz="0 -${table_width} 0"/>
-    <xacro:table_module table_id="$(arg table_2_name)" connected_to="$(arg table_0_name)" xyz="0 ${table_width} 0"/>
-    <xacro:table_module table_id="$(arg table_3_name)" connected_to="$(arg table_0_name)" xyz="-${table_width} 0 0"/>
-    <xacro:table_module table_id="$(arg table_4_name)" connected_to="$(arg table_3_name)" xyz="0 -${table_width} 0"/>
-    <xacro:table_module table_id="$(arg table_5_name)" connected_to="$(arg table_3_name)" xyz="0 ${table_width} 0"/>
+    <xacro:table_module table_id="$(arg table_0_name)" connected_to="world" xyz="0 0 ${table_height}" rpy="0 0 0"/>
+    <xacro:table_module table_id="$(arg table_1_name)" connected_to="$(arg table_0_name)" xyz="0 -${table_width} 0" rpy="0 0 0"/>
+    <xacro:table_module table_id="$(arg table_2_name)" connected_to="$(arg table_0_name)" xyz="0 ${table_width} 0" rpy="0 0 0"/>
+    <xacro:table_module table_id="$(arg table_3_name)" connected_to="$(arg table_0_name)" xyz="-${table_width} 0 0" rpy="0 0 0"/>
+    <xacro:table_module table_id="$(arg table_4_name)" connected_to="$(arg table_3_name)" xyz="0 -${table_width} 0" rpy="0 0 0"/>
+    <xacro:table_module table_id="$(arg table_5_name)" connected_to="$(arg table_3_name)" xyz="0 ${table_width} 0" rpy="0 0 1.57"/>
     <!-- <xacro:table_module table_id="$(arg table_6_name)" connected_to="$(arg table_5_name)" xyz="-${table_width} 0 0"/>-->
     <xacro:vise_setup connected_to="$(arg table_3_name)" xyz="0 0 0"/>

File: reconcycle_description/urdf/table_module.xacro (robot description, xacro)
@@ -1,5 +1,5 @@
 <?xml version='1.0'?>
 <robot xmlns:xacro="http://www.ros.org/wiki/xacro" name="table_module">
-<xacro:macro name="table_module" params="table_id:='table' connected_to:='' xyz:=''">
+<xacro:macro name="table_module" params="table_id:='table' connected_to:='' xyz:='' rpy:=''">
     <xacro:unless value="${not connected_to}">
       <joint name="${table_id}_joint_${connected_to}" type="fixed">
@@ -7,5 +7,5 @@
         <child link="${table_id}"/>
         <xacro:unless value="${not xyz}">
-            <origin rpy="0 0 0" xyz="${xyz}"/>
+            <origin rpy="${rpy}" xyz="${xyz}"/>
         </xacro:unless>
         <xacro:if value="${not xyz}">
