Commit message: Urdf changes.

File: reconcycle_description/urdf/cuboid_layout.urdf (robot description, URDF)
Before this commit: robot cuboid, 1 links, 0 joints
Links:
- removed link cuboid
- added link cuboid_link, mass 0.2; collision mesh filename=package://reconcycle_description/meshes/cuboid.obj scale=1 1 1; visual mesh filename=package://reconcycle_description/meshes/cuboid.obj scale=1 1 1

Commit message: xacro and urdf files modifications.

File: reconcycle_description/urdf/cuboid_layout.urdf (robot description, URDF)
Before this commit: robot cuboid, 1 links, 0 joints
Links:
- link cuboid_link: geometry collision cylinder length=0.75 radius=0.07; visual cylinder length=0.75 radius=0.07

File: reconcycle_description/urdf/cuboid_layout.xacro (robot description, xacro)
@@ -1,5 +1,5 @@
 <?xml version="1.0"?>
 <robot xmlns:xacro="http://www.ros.org/wiki/xacro" name="cuboid">
-    <link name="cuboid">
+    <link name="cuboid_link">
         <visual>
             <origin rpy="0 0 0" xyz=" 0 0 0 "/>
