Commit message: Mass and inertia values.

File: reconcycle_description/urdf/cuboid_layout.xacro (robot description, xacro)
@@ -14,6 +14,6 @@
     <inertial>
         <origin xyz="0 0 0" rpy="0 0 0"/>
-        <mass value="20"/>
-        <inertia ixx="20" ixy="0.0" ixz="0.0" iyy="20" iyz="0.0" izz="20"/>
+        <mass value="0.2"/>
+        <inertia ixx="2" ixy="0.0" ixz="0.0" iyy="2" iyz="0.0" izz="2"/>
     </inertial>
 </link>

Commit message: Urdf file changes

File: reconcycle_description/urdf/cuboid_layout.xacro (robot description, xacro)
@@ -1,19 +1,27 @@
-<link name="cuboid">
-    <visual>
-        <origin rpy="0 0 0" xyz=" 0 0 0 "/>
-        <geometry>
-            <mesh filename="package://reconcycle_description/meshes/cuboid.obj" scale="0.001 0.001 0.001"/>
-        </geometry>
-    </visual>
-    <collision>
-        <origin rpy="0 0 0" xyz="0.0 0.0 0"/>
-        <geometry>
-            <mesh filename="package://reconcycle_description/meshes/cuboid.obj" scale="0.001 0.001 0.001"/>
-        </geometry>
-    </collision>
-    <inertial>
-        <origin xyz="0 0 0" rpy="0 0 0"/>
-        <mass value="0.2"/>
-        <inertia ixx="2" ixy="0.0" ixz="0.0" iyy="2" iyz="0.0" izz="2"/>
-    </inertial>
-</link>
+<?xml version="1.0"?>
+<robot xmlns:xacro="http://www.ros.org/wiki/xacro" name="cuboid">
+    <link name="cuboid">
+        <visual>
+            <origin rpy="0 0 0" xyz=" 0 0 0 "/>
+            <geometry>
+                <mesh filename="package://reconcycle_description/meshes/cuboid.obj" scale="1 1 1"/>
+            </geometry>
+        </visual>
+        <collision>
+            <origin rpy="0 0 0" xyz="0.0 0.0 0"/>
+            <geometry>
+                <mesh filename="package://reconcycle_description/meshes/cuboid.obj" scale="1 1 1"/>
+            </geometry>
+        </collision>
+        <inertial>
+            <origin xyz="0 0 0" rpy="0 0 0"/>
+            <mass value="0.2"/>
+            <inertia ixx="2" ixy="0.0" ixz="0.0" iyy="2" iyz="0.0" izz="2"/>
+        </inertial>
+    </link>
+    <gazebo>
+        <plugin name="control" filename="libgazebo_ros_control.so">
+            <robotNamespace>cuboid</robotNamespace>
+        </plugin>
+    </gazebo>
+</robot>

Commit message: Add scaling for correct visualization

File: reconcycle_description/urdf/cuboid_layout.xacro (robot description, xacro)
@@ -5,5 +5,5 @@
             <origin rpy="0 0 0" xyz=" 0 0 0 "/>
             <geometry>
-                <mesh filename="package://reconcycle_description/meshes/cuboid.obj" scale="1 1 1"/>
+                <mesh filename="package://reconcycle_description/meshes/cuboid.obj" scale="0.01 0.01 0.01"/>
             </geometry>
         </visual>
@@ -11,5 +11,5 @@
             <origin rpy="0 0 0" xyz="0.0 0.0 0"/>
             <geometry>
-                <mesh filename="package://reconcycle_description/meshes/cuboid.obj" scale="1 1 1"/>
+                <mesh filename="package://reconcycle_description/meshes/cuboid.obj" scale="0.01 0.01 0.01"/>
             </geometry>
         </collision>

Commit message: Add red material on cuboid for better visibility on gray table.

File: reconcycle_description/urdf/cuboid_layout.xacro (robot description, xacro)
@@ -1,15 +1,19 @@
 <?xml version="1.0"?>
 <robot xmlns:xacro="http://www.ros.org/wiki/xacro" name="cuboid">
+    <material name="red">
+        <color rgba="1.0 0.0 0.0 1.0"/>
+    </material>
     <link name="cuboid_link">
         <visual>
             <origin rpy="0 0 0" xyz=" 0 0 0 "/>
             <geometry>
-                <mesh filename="package://reconcycle_description/meshes/cuboid.obj" scale="0.01 0.01 0.01"/>
+                <mesh filename="package://reconcycle_description/meshes/cuboid.stl" scale="0.01 0.01 0.01"/>
             </geometry>
+            <material name="red"/>
         </visual>
         <collision>
             <origin rpy="0 0 0" xyz="0.0 0.0 0"/>
             <geometry>
-                <mesh filename="package://reconcycle_description/meshes/cuboid.obj" scale="0.01 0.01 0.01"/>
+                <mesh filename="package://reconcycle_description/meshes/cuboid.stl" scale="0.01 0.01 0.01"/>
             </geometry>
         </collision>
