Commit message: Model name change in xacro, updated rviz view

File: reconcycle_description/urdf/reconcycle_default_models.xacro (robot description, xacro)
@@ -206,11 +206,11 @@
                 <origin rpy="${pi/2} 0 0" xyz=" 0 0 0 "/>
                 <geometry>
-                    <mesh filename="package://reconcycle_description/meshes/tools_setup.obj" scale="0.001 0.001 0.001"/>
-                </geometry>
-            </visual>
-            <collision>
-                <origin rpy="${pi/2} 0 0" xyz="0.0 0.0 0"/>
-                <geometry>
-                    <mesh filename="package://reconcycle_description/meshes/tools_setup.obj" scale ="0.001 0.001 0.001"/>
+                    <mesh filename="package://reconcycle_description/meshes/toolholder_setup.obj" scale="0.001 0.001 0.001"/>
+                </geometry>
+            </visual>
+            <collision>
+                <origin rpy="${pi/2} 0 0" xyz="0.0 0.0 0"/>
+                <geometry>
+                    <mesh filename="package://reconcycle_description/meshes/toolholder_setup.obj" scale ="0.001 0.001 0.001"/>
                 </geometry>
             </collision>
