Commit message: Added flange

File: reconcycle_description/urdf/hca_layout.xacro (robot description, xacro)
@@ -21,3 +21,4 @@
     <xacro:table_module table_id="$(arg table_5_name)" connected_to="$(arg table_3_name)" xyz="0 ${table_width} 0"/>
     <xacro:table_module table_id="$(arg table_6_name)" connected_to="$(arg table_5_name)" xyz="-${table_width} 0 0"/>
+    <xacro:vise_setup connected_to="$(arg table_3_name)" xyz="0 0 0"/>
 </robot>

File: reconcycle_description/urdf/reconcycle_defaults.xacro (robot description, xacro)
@@ -5,4 +5,5 @@
 <xacro:property name="table_height" value="0.805" />
 <xacro:arg name="table_surf_thickness" default="0.02"/>
+<xacro:property name="flange_thickness" value="0.01"/>
 <xacro:macro name="tc_tool_side" params="tc_id:='tc_tool_1' connected_to:='' xyz:='0 0 0' rpy='0 0 0'">
     <!--  If connected_to is not provided we don't do anything -->
@@ -66,3 +67,66 @@
     </xacro:unless>
 </xacro:macro>
+<!-- Robot flange -->
+<xacro:macro name="flange" params="flange_id:='flange' connected_to:='' xyz:='0 0 0' rpy='0 0 0'">
+    <!--  If connected_to is not provided we don't do anything -->
+    <xacro:unless value="${not connected_to}">
+        <joint name="${flange_id}_joint_${connected_to}" type="fixed">
+            <parent link="${connected_to}"/>
+            <child link="${flange_id}"/>
+            <origin rpy="${rpy}" xyz="${xyz}"/>
+            <dynamics damping="1"/>
+        </joint>
+        <!-- The tool changer -->
+        <link name="${flange_id}">
+            <visual>
+                <origin rpy="${pi/2} 0 0" xyz=" 0 0 0 "/>
+                <geometry>
+                    <mesh filename="package://reconcycle_description/meshes/flange.obj" scale="0.001 0.001 0.001"/>
+                </geometry>
+            </visual>
+            <collision>
+                <origin rpy="${pi/2} 0 0" xyz="0.0 0.0 0"/>
+                <geometry>
+                    <mesh filename="package://reconcycle_description/meshes/flange.obj" scale ="0.001 0.001 0.001"/>
+                </geometry>
+            </collision>
+            <inertial>
+                <origin xyz="0 0 0" rpy="0 0 0"/>
+                <mass value="0.07"/>
+                <inertia ixx="0.07" ixy="0.0" ixz="0.0" iyy="0.07" iyz="0.0" izz="0.07"/>
+            </inertial>
+        </link>
+    </xacro:unless>
+</xacro:macro>
+<xacro:macro name="vise_setup" params="vise_id:='vise' connected_to:='' xyz:='0 0 0' rpy='0 0 0'">
+    <!--  If connected_to is not provided we don't do anything -->
+    <xacro:unless value="${not connected_to}">
+        <joint name="${vise_id}_joint_${connected_to}" type="fixed">
+            <parent link="${connected_to}"/>
+            <child link="${vise_id}"/>
+            <origin rpy="${rpy}" xyz="${xyz}"/>
+            <dynamics damping="1"/>
+        </joint>
+        <!-- The vise -->
+        <link name="${vise_id}">
+            <visual>
+                <origin rpy="${pi/2} 0 0" xyz=" 0 0 0 "/>
+                <geometry>
+                    <mesh filename="package://reconcycle_description/meshes/vise_setup.obj" scale="0.001 0.001 0.001"/>
+                </geometry>
+            </visual>
+            <collision>
+                <origin rpy="${pi/2} 0 0" xyz="0.0 0.0 0"/>
+                <geometry>
+                    <mesh filename="package://reconcycle_description/meshes/vise_setup.obj" scale ="0.001 0.001 0.001"/>
+                </geometry>
+            </collision>
+            <inertial>
+                <origin xyz="0 0 0" rpy="0 0 0"/>
+                <mass value="3"/>
+                <inertia ixx="3.0" ixy="0.0" ixz="0.0" iyy="3.0" iyz="0.0" izz="3.0"/>
+            </inertial>
+        </link>
+    </xacro:unless>
+</xacro:macro>
 </robot>

File: reconcycle_description/urdf/reconcycle_panda.xacro (robot description, xacro)
@@ -12,5 +12,7 @@
     <!-- Call the macro -->
     <xacro:panda_robot load_gazebo="$(arg load_gazebo)" robot_name="$(arg robot_name)" connected_to="$(arg robot_name)"/>
+    <!-- Attach the flange to the robot -->
+    <xacro:flange flange_id="$(arg robot_name)_flange" connected_to="$(arg robot_name)_link8"/>
     <!-- Attach the tool exchange to the robot -->
-    <xacro:tc_robot_side tc_id="$(arg robot_name)_tc_robot" connected_to="$(arg robot_name)_link8"/>
+    <xacro:tc_robot_side tc_id="$(arg robot_name)_tc_robot" connected_to="$(arg robot_name)_flange" xyz="0 0 ${flange_thickness}"/>
 </robot>

Commit message: Added frames to tool holder - tool_frame_#NUM

File: reconcycle_description/urdf/hca_layout.xacro (robot description, xacro)
@@ -25,3 +25,7 @@
     <xacro:cutter_model connected_to="$(arg table_6_name)" xyz="0 0 0" />
     <xacro:tool_model connected_to="$(arg table_2_name)" xyz="0 0 0" />
+    <xacro:tool_frame_1 connected_to="$(arg table_2_name)" xyz="0.18 -0.036 0.355" rpy="0 3.1415 0" />
+    <xacro:tool_frame_2 connected_to="$(arg table_2_name)" xyz="0.06 -0.036 0.355" rpy="0 3.1415 0" />
+    <xacro:tool_frame_3 connected_to="$(arg table_2_name)" xyz="-0.06 -0.036 0.355" rpy="0 3.1415 0" />
+    <xacro:tool_frame_4 connected_to="$(arg table_2_name)" xyz="-0.18 -0.036 0.355" rpy="0 3.1415 0" />
 </robot>

File: reconcycle_description/urdf/reconcycle_default_models.xacro (robot description, xacro)
@@ -223,3 +223,127 @@
     </xacro:unless>
 </xacro:macro>
+<xacro:macro name="tool_frame_1" params="tool_id:='tool_frame_1' connected_to:='' xyz:='0.0 0.0 0.0' rpy='0 0 0'">
+    <!--  If connected_to is not provided we don't do anything -->
+    <xacro:unless value="${not connected_to}">
+        <joint name="${tool_id}_joint_${connected_to}" type="fixed">
+            <parent link="${connected_to}"/>
+            <child link="${tool_id}"/>
+            <origin rpy="${rpy}" xyz="${xyz}"/>
+            <dynamics damping="1"/>
+        </joint>
+        <!-- The vise -->
+        <link name="${tool_id}">
+            <visual>
+                <origin rpy="${pi/2} 0 0" xyz=" 0 0 0 "/>
+                <geometry>
+                    <mesh filename="package://reconcycle_description/meshes/EmptyCubeFrame.obj" scale="0.001 0.001 0.001"/>
+                </geometry>
+            </visual>
+            <collision>
+                <origin rpy="${pi/2} 0 0" xyz="0.0 0.0 0"/>
+                <geometry>
+                    <mesh filename="package://reconcycle_description/meshes/EmptyCubeFrame.obj" scale ="0.001 0.001 0.001"/>
+                </geometry>
+            </collision>
+            <inertial>
+                <origin xyz="0 0 0" rpy="0 0 0"/>
+                <mass value="3"/>
+                <inertia ixx="3.0" ixy="0.0" ixz="0.0" iyy="3.0" iyz="0.0" izz="3.0"/>
+            </inertial>
+        </link>
+    </xacro:unless>
+</xacro:macro>
+<xacro:macro name="tool_frame_2" params="tool_id:='tool_frame_2' connected_to:='' xyz:='0.0 0.0 0.0' rpy='0 0 0'">
+    <!--  If connected_to is not provided we don't do anything -->
+    <xacro:unless value="${not connected_to}">
+        <joint name="${tool_id}_joint_${connected_to}" type="fixed">
+            <parent link="${connected_to}"/>
+            <child link="${tool_id}"/>
+            <origin rpy="${rpy}" xyz="${xyz}"/>
+            <dynamics damping="1"/>
+        </joint>
+        <!-- The vise -->
+        <link name="${tool_id}">
+            <visual>
+                <origin rpy="${pi/2} 0 0" xyz=" 0 0 0 "/>
+                <geometry>
+                    <mesh filename="package://reconcycle_description/meshes/EmptyCubeFrame.obj" scale="0.001 0.001 0.001"/>
+                </geometry>
+            </visual>
+            <collision>
+                <origin rpy="${pi/2} 0 0" xyz="0.0 0.0 0"/>
+                <geometry>
+                    <mesh filename="package://reconcycle_description/meshes/EmptyCubeFrame.obj" scale ="0.001 0.001 0.001"/>
+                </geometry>
+            </collision>
+            <inertial>
+                <origin xyz="0 0 0" rpy="0 0 0"/>
+                <mass value="3"/>
+                <inertia ixx="3.0" ixy="0.0" ixz="0.0" iyy="3.0" iyz="0.0" izz="3.0"/>
+            </inertial>
+        </link>
+    </xacro:unless>
+</xacro:macro>
+<xacro:macro name="tool_frame_3" params="tool_id:='tool_frame_3' connected_to:='' xyz:='0.0 0.0 0.0' rpy='0 0 0'">
+    <!--  If connected_to is not provided we don't do anything -->
+    <xacro:unless value="${not connected_to}">
+        <joint name="${tool_id}_joint_${connected_to}" type="fixed">
+            <parent link="${connected_to}"/>
+            <child link="${tool_id}"/>
+            <origin rpy="${rpy}" xyz="${xyz}"/>
+            <dynamics damping="1"/>
+        </joint>
+        <!-- The vise -->
+        <link name="${tool_id}">
+            <visual>
+                <origin rpy="${pi/2} 0 0" xyz=" 0 0 0 "/>
+                <geometry>
+                    <mesh filename="package://reconcycle_description/meshes/EmptyCubeFrame.obj" scale="0.001 0.001 0.001"/>
+                </geometry>
+            </visual>
+            <collision>
+                <origin rpy="${pi/2} 0 0" xyz="0.0 0.0 0"/>
+                <geometry>
+                    <mesh filename="package://reconcycle_description/meshes/EmptyCubeFrame.obj" scale ="0.001 0.001 0.001"/>
+                </geometry>
+            </collision>
+            <inertial>
+                <origin xyz="0 0 0" rpy="0 0 0"/>
+                <mass value="3"/>
+                <inertia ixx="3.0" ixy="0.0" ixz="0.0" iyy="3.0" iyz="0.0" izz="3.0"/>
+            </inertial>
+        </link>
+    </xacro:unless>
+</xacro:macro>
+<xacro:macro name="tool_frame_4" params="tool_id:='tool_frame_4' connected_to:='' xyz:='0.0 0.0 0.0' rpy='0 0 0'">
+    <!--  If connected_to is not provided we don't do anything -->
+    <xacro:unless value="${not connected_to}">
+        <joint name="${tool_id}_joint_${connected_to}" type="fixed">
+            <parent link="${connected_to}"/>
+            <child link="${tool_id}"/>
+            <origin rpy="${rpy}" xyz="${xyz}"/>
+            <dynamics damping="1"/>
+        </joint>
+        <!-- The vise -->
+        <link name="${tool_id}">
+            <visual>
+                <origin rpy="${pi/2} 0 0" xyz=" 0 0 0 "/>
+                <geometry>
+                    <mesh filename="package://reconcycle_description/meshes/EmptyCubeFrame.obj" scale="0.001 0.001 0.001"/>
+                </geometry>
+            </visual>
+            <collision>
+                <origin rpy="${pi/2} 0 0" xyz="0.0 0.0 0"/>
+                <geometry>
+                    <mesh filename="package://reconcycle_description/meshes/EmptyCubeFrame.obj" scale ="0.001 0.001 0.001"/>
+                </geometry>
+            </collision>
+            <inertial>
+                <origin xyz="0 0 0" rpy="0 0 0"/>
+                <mass value="3"/>
+                <inertia ixx="3.0" ixy="0.0" ixz="0.0" iyy="3.0" iyz="0.0" izz="3.0"/>
+            </inertial>
+        </link>
+    </xacro:unless>
+</xacro:macro>
 </robot>
