Commit message: Update

File: reconcycle_description/urdf/tc_robot_side.xacro (robot description, xacro)
@@ -3,5 +3,5 @@
     <link name="tc_robot">
         <visual>
-            <origin rpy="1.57 0 0" xyz=" 0 0 0 "/>
+            <origin rpy="1.57 0 -0.802664626" xyz=" 0 0 0 "/>
             <geometry>
                 <mesh filename="package://reconcycle_description/meshes/tc_robot_side.obj" scale="0.001 0.001 0.001"/>
@@ -9,5 +9,5 @@
         </visual>
         <collision>
-            <origin rpy="1.57 0 0" xyz="0.0 0.0 0"/>
+            <origin rpy="1.57 0 -0.802664626" xyz="0.0 0.0 0"/>
             <geometry>
                 <mesh filename="package://reconcycle_description/meshes/tc_robot_side.obj" scale ="0.001 0.001 0.001"/>

Commit message: fixed missing connections in tf tree

File: reconcycle_description/urdf/tc_robot_side.xacro (robot description, xacro)
@@ -1,5 +1,6 @@
 <?xml version='1.0'?>
 <robot xmlns:xacro="http://www.ros.org/wiki/xacro" name="defaults">
-    <link name="tc_robot">
+<xacro:macro name = "tc_robot" param="tc_id:='tc_robot' connected_to:='panda_link8'" >
+    <link name="${tc_id}">
         <visual>
             <origin rpy="1.57 0 -0.802664626" xyz=" 0 0 0 "/>
@@ -20,3 +21,8 @@
         </inertial>
     </link>
+    <joint name="${tc_id}" type="fixed">
+        <parent link="${connected_to}"/>
+        <child link="${tc_id}"/>
+    </joint>
+</xacro:macro>
 </robot>
