Commit message: vise stil not good

File: reconcycle_description/urdf/vise_desk.urdf (robot description, URDF)
Before this commit: robot fifi, 10 links, 9 joints
Links:
- added link viseOne; visual mesh filename=package://test_rospkg/meshes/vise_desk/RCY-003-012-040.stl; visual mesh filename=package://test_rospkg/meshes/vise_desk/RCY-003-013-0040.stl
- added link viseTw
- added link viseTwo; visual mesh filename=package://test_rospkg/meshes/vise_desk/SOLID45.stl; visual mesh filename=package://test_rospkg/meshes/vise_desk/WJ200UM_01_10_20.stl
- link base: geometry visual mesh filename=package://test_rospkg/meshes/vise_desk/095-000-002-DIN63210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; visual mesh filename=package://test_rospkg/meshes/vise_desk/095-000-002-DIN63211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
- link viseOn: geometry visual mesh filename=package://test_rospkg/meshes/vise_desk/RCY-003-013-0041.stl; visual mesh filename=package://test_rospkg/meshes/vise_desk/SOLID48.stl
Joints:
- added joint base_viseOne: type prismatic, parent base, child viseOne, origin xyz=0.35220447066381433 0.32190952633305603 0.05995923113227309 rpy=3.1415926535897696 1.5707963267948966 0.0, axis 0 0 1, limit lower=-1.548 upper=1.548 effort=1000 velocity=0.5
- added joint base_viseTw: type prismatic, parent base, child viseTw, origin xyz=0.2812044706638224 0.3644095263330476 0.02095923113227434 rpy=3.141592653589793 1.5707963267948617 1.5755657659879256, axis 0 0 1, limit lower=-1.548 upper=1.548 effort=1000 velocity=0.5
- added joint base_viseTwo: type prismatic, parent base, child viseTwo, origin xyz=0.3212044706638124 0.2394095263330476 0.020959231122270352 rpy=1.0090602588783764 1.5707963267948308 2.5812047513500547, axis 0 0 1, limit lower=-1.548 upper=1.548 effort=1000 velocity=0.5
