Commit message: update models but dont add .stls

File: reconcycle_description/urdf/cutter.urdf (robot description, URDF)
Before this commit: robot fifi, 14 links, 13 joints
Links:
- link base: geometry visual mesh filename=package://reconcycle_description/meshes/cutter/095-000-002-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; visual mesh filename=package://reconcycle_description/meshes/cutter/095-000-002-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

File: reconcycle_description/urdf/vise_desk.urdf (robot description, URDF)
Before this commit: robot fifi, 13 links, 12 joints
Links:
- removed link viseOn
- removed link viseTw
- added link viseOne1; visual mesh filename=package://reconcycle_description/meshes/vise_desk/RCY-003-0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; visual mesh filename=package://reconcycle_description/meshes/vise_desk/SOLID47.s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
- added link viseTwo1; visual mesh filename=package://reconcycle_description/meshes/vise_desk/SOLID46.s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; visual mesh filename=package://reconcycle_description/meshes/vise_desk/WJ200UM_0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
- link viseOne: geometry visual mesh filename=package://reconcycle_description/meshes/vise_desk/RCY-003-0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; visual mesh filename=package://reconcycle_description/meshes/vise_desk/RCY-003-0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
Joints:
- removed joint base_viseOn
- removed joint base_viseTw
- added joint base_viseOne1: type prismatic, parent base, child viseOne1, origin xyz=0.42900000000000027 0.2600000000000093 0.1089592311322698 rpy=3.1415926535897696 1.5707963267948966 0.0, axis 0 0 1, limit lower=-1.548 upper=1.548 effort=1000 velocity=0.5
- added joint base_viseTwo1: type prismatic, parent base, child viseTwo1, origin xyz=0.39800000000000074 0.17649999999999993 0.06995923113226832 rpy=0.018985060498840408 1.5707963267948615 1.5929446032344046, axis 0 0 1, limit lower=-1.548 upper=1.548 effort=1000 velocity=0.5
- joint base_viseOne: origin xyz=0.35220447066381433 0.32190952633305603 0.05995923113227309 rpy=3.1415926535897696 1.5707963267948966 0.0 -> xyz=0.327000000000001 0.21999999999999914 0.10895923112226945 rpy=1.5707963267948966 1.5707963267948608 1.5707963267949052
- joint base_viseTwo: origin xyz=0.3212044706638124 0.2394095263330476 0.020959231122270352 rpy=1.0090602588783764 1.5707963267948308 2.5812047513500547 -> xyz=0.3580000000000007 0.3035000000000004 0.06995923113227184 rpy=3.1179377606468486 1.5707963267948615 1.5486480503553888
