Commit message: merged robot_cell_description into reconcycle_description

File: reconcycle_description/urdf/reconcycle_generic.urdf.xacro (robot description, xacro)
@@ -1,4 +1,4 @@
 <?xml version="1.0"?>
-<robot xmlns:xacro="http://www.ros.org/wiki/xacro"  name="robot_cell">
+<robot xmlns:xacro="http://www.ros.org/wiki/xacro"  name="reconcycle_generic">
   <xacro:macro name="loop_code" params="current_i names_vector yaml_data_dictionary"  >
     <xacro:property name="current_name" value="${names_vector[current_i]}"/>
@@ -24,5 +24,5 @@
   </xacro:macro>
   <!-- ACTUAL PROGRAM-->
-  <xacro:property name="yaml_file" value="$(find robot_cell_description)/config/active_config.yaml" />
+  <xacro:property name="yaml_file" value="$(find reconcycle_description)/config/active_config.yaml" />
   <xacro:property name="active_config" value="${xacro.load_yaml(yaml_file)}"/>
   <xacro:property name="list_of_active_elements_names" value="${active_config['active_description_elements']}"/>

Commit message: ifam 2024 settings

File: reconcycle_description/urdf/reconcycle_generic.urdf.xacro (robot description, xacro)
@@ -9,5 +9,5 @@
         <origin xyz="${yaml_data_dictionary[current_name]['x']} ${yaml_data_dictionary[current_name]['y']} ${yaml_data_dictionary[current_name]['z']}" rpy="${yaml_data_dictionary[current_name]['er']} ${yaml_data_dictionary[current_name]['ep']} ${yaml_data_dictionary[current_name]['ey']}" />
         <axis xyz="1 0 0"/>
-        <parent link="${yaml_data_dictionary[current_name]['parrent']}"/>
+        <parent link="${yaml_data_dictionary[current_name]['parent']}"/>
         <child link="${this_robot_name + 'base'}"/>
     </joint>
@@ -27,5 +27,5 @@
   <xacro:property name="active_config" value="${xacro.load_yaml(yaml_file)}"/>
   <xacro:property name="list_of_active_elements_names" value="${active_config['active_description_elements']}"/>
-  <link name="robot_cell_base">
+  <link name="reconcycle_base">
   </link>
   <xacro:loop current_i="${len(list_of_active_elements_names)}" names_vector = "${list_of_active_elements_names}" yaml_data_dictionary="${active_config}"/>
