Commit message: correct tf mappings

File: reconcycle_description/urdf/schunk_pzh20.xacro (robot description, xacro)
@@ -1,4 +1,7 @@
 <?xml version='1.0'?>
 <robot xmlns:xacro="http://www.ros.org/wiki/xacro" name="schunk_pzh20_gripper">
+    <material name="white">
+        <color rgba="1 1 1 1"/>
+    </material>
     <xacro:arg name="schunk_gripper_id" default="schunk_pzh20"/>
     <link name="$(arg schunk_gripper_id)">
@@ -8,4 +11,5 @@
                 <mesh filename="package://reconcycle_description/meshes/grippers/schunk_pzh20.stl" scale="0.001 0.001 0.001"/>
             </geometry>
+            <material name="white"/>
         </visual>
         <collision>

File: reconcycle_description/urdf/schunk_pzh20_adapter.xacro (robot description, xacro)
@@ -1,4 +1,7 @@
 <?xml version='1.0'?>
 <robot xmlns:xacro="http://www.ros.org/wiki/xacro" name="schunk_pzh20_adapter">
+    <material name="darkgray">
+        <color rgba="0.5 0.5 0.5 0.8"/>
+    </material>
     <xacro:arg name="schunk_adapter_id" default="schunk_pzh20_adapter"/>
     <link name="$(arg schunk_adapter_id)">
@@ -8,4 +11,5 @@
                 <mesh filename="package://reconcycle_description/meshes/grippers/schunk_to_tc_adapter.stl" scale="0.001 0.001 0.001"/>
             </geometry>
+            <material name="darkgray"/>
         </visual>
         <collision>
