Commit message: added rvizweb config

File: reconcycle_description/urdf/reconcycle_defaults.xacro (robot description, xacro)
@@ -19,5 +19,5 @@
                 <origin rpy="$0 0 0" xyz=" 0 0 0 "/>
                 <geometry>
-                    <mesh filename="package://reconcycle_description/meshes/tc_tool_side.obj" scale="0.001 0.001 0.001"/>
+                    <mesh filename="package://reconcycle_description/meshes/tc_tool_side.dae" scale="0.001 0.001 0.001"/>
                 </geometry>
             </visual>
@@ -25,5 +25,5 @@
                 <origin rpy="${pi/2} 0 0" xyz="0.0 0.0 0"/>
                 <geometry>
-                    <mesh filename="package://reconcycle_description/meshes/tc_tool_side.obj" scale ="0.001 0.001 0.001"/>
+                    <mesh filename="package://reconcycle_description/meshes/tc_tool_side.dae" scale ="0.001 0.001 0.001"/>
                 </geometry>
             </collision>
@@ -50,5 +50,5 @@
                 <origin rpy="${-pi/2} 0 0" xyz=" 0 0 0 "/>
                 <geometry>
-                    <mesh filename="package://reconcycle_description/meshes/tc_robot_side.obj" scale="0.001 0.001 0.001"/>
+                    <mesh filename="package://reconcycle_description/meshes/tc_robot_side.dae" scale="0.001 0.001 0.001"/>
                 </geometry>
             </visual>
@@ -56,5 +56,5 @@
                 <origin rpy="${-pi/2} 0 0" xyz="0.0 0.0 0"/>
                 <geometry>
-                    <mesh filename="package://reconcycle_description/meshes/tc_robot_side.obj" scale ="0.001 0.001 0.001"/>
+                    <mesh filename="package://reconcycle_description/meshes/tc_robot_side.dae" scale ="0.001 0.001 0.001"/>
                 </geometry>
             </collision>
@@ -82,5 +82,5 @@
                 <origin rpy="${pi/2} 0 0" xyz=" 0 0 0 "/>
                 <geometry>
-                    <mesh filename="package://reconcycle_description/meshes/flange.obj" scale="0.001 0.001 0.001"/>
+                    <mesh filename="package://reconcycle_description/meshes/flange.dae" scale="0.001 0.001 0.001"/>
                 </geometry>
             </visual>
@@ -88,5 +88,5 @@
                 <origin rpy="${pi/2} 0 0" xyz="0.0 0.0 0"/>
                 <geometry>
-                    <mesh filename="package://reconcycle_description/meshes/flange.obj" scale ="0.001 0.001 0.001"/>
+                    <mesh filename="package://reconcycle_description/meshes/flange.dae" scale ="0.001 0.001 0.001"/>
                 </geometry>
             </collision>
@@ -113,5 +113,5 @@
                 <origin rpy="${pi/2} 0 0" xyz=" 0 0 0 "/>
                 <geometry>
-                    <mesh filename="package://reconcycle_description/meshes/vise_setup.obj" scale="0.001 0.001 0.001"/>
+                    <mesh filename="package://reconcycle_description/meshes/vise_setup.dae" scale="0.001 0.001 0.001"/>
                 </geometry>
             </visual>
@@ -119,5 +119,5 @@
                 <origin rpy="${pi/2} 0 0" xyz="0.0 0.0 0"/>
                 <geometry>
-                    <mesh filename="package://reconcycle_description/meshes/vise_setup.obj" scale ="0.001 0.001 0.001"/>
+                    <mesh filename="package://reconcycle_description/meshes/vise_setup.dae" scale ="0.001 0.001 0.001"/>
                 </geometry>
             </collision>

Commit message: added vise_base to reconcycle_defaults.xacro

File: reconcycle_description/urdf/reconcycle_defaults.xacro (robot description, xacro)
@@ -347,3 +347,34 @@
     </xacro:unless>
 </xacro:macro>
+<xacro:macro name="vise_base" params="vise_id:='vise_base' connected_to:='' xyz:='0 0 0' rpy='0 0 0'">
+    <!--  If connected_to is not provided we don't do anything -->
+    <xacro:unless value="${not connected_to}">
+        <joint name="${vise_id}_joint_${connected_to}" type="fixed">
+            <parent link="${connected_to}"/>
+            <child link="${vise_id}"/>
+            <origin rpy="${rpy}" xyz="${xyz}"/>
+            <dynamics damping="1"/>
+        </joint>
+        <!-- The vise -->
+        <link name="${vise_id}">
+            <visual>
+                <origin rpy="${pi/2} 0 0" xyz=" 0 0 0 "/>
+                <geometry>
+                    <mesh filename="package://reconcycle_description/meshes/vise_base.obj" scale="0.001 0.001 0.001"/>
+                </geometry>
+            </visual>
+            <collision>
+                <origin rpy="${pi/2} 0 0" xyz="0.0 0.0 0"/>
+                <geometry>
+                    <mesh filename="package://reconcycle_description/meshes/vise_base.obj" scale ="0.001 0.001 0.001"/>
+                </geometry>
+            </collision>
+            <inertial>
+                <origin xyz="0 0 0" rpy="0 0 0"/>
+                <mass value="3"/>
+                <inertia ixx="3.0" ixy="0.0" ixz="0.0" iyy="3.0" iyz="0.0" izz="3.0"/>
+            </inertial>
+        </link>
+    </xacro:unless>
+</xacro:macro>
 </robot>

Commit message: added cutter_base to xacro

File: reconcycle_description/urdf/reconcycle_defaults.xacro (robot description, xacro)
@@ -378,3 +378,34 @@
     </xacro:unless>
 </xacro:macro>
+<xacro:macro name="cutter_base" params="cutter_id:='cutter_base' connected_to:='' xyz:='0 0 0' rpy='0 0 0'">
+    <!--  If connected_to is not provided we don't do anything -->
+    <xacro:unless value="${not connected_to}">
+        <joint name="${cutter_id}_joint_${connected_to}" type="fixed">
+            <parent link="${connected_to}"/>
+            <child link="${cutter_id}"/>
+            <origin rpy="${rpy}" xyz="${xyz}"/>
+            <dynamics damping="1"/>
+        </joint>
+        <!-- The vise -->
+        <link name="${cutter_id}">
+            <visual>
+                <origin rpy="${pi/2} 0 0" xyz=" 0 0 0 "/>
+                <geometry>
+                    <mesh filename="package://reconcycle_description/meshes/pneumatic_cutter_base.obj" scale="0.001 0.001 0.001"/>
+                </geometry>
+            </visual>
+            <collision>
+                <origin rpy="${pi/2} 0 0" xyz="0.0 0.0 0"/>
+                <geometry>
+                    <mesh filename="package://reconcycle_description/meshes/pneumatic_cutter_base.obj" scale ="0.001 0.001 0.001"/>
+                </geometry>
+            </collision>
+            <inertial>
+                <origin xyz="0 0 0" rpy="0 0 0"/>
+                <mass value="3"/>
+                <inertia ixx="3.0" ixy="0.0" ixz="0.0" iyy="3.0" iyz="0.0" izz="3.0"/>
+            </inertial>
+        </link>
+    </xacro:unless>
+</xacro:macro>
 </robot>

Commit message: cleanup

File: reconcycle_description/urdf/reconcycle_defaults.xacro (robot description, xacro)
@@ -17,5 +17,5 @@
         <link name="${tc_id}">
             <visual>
-                <origin rpy="$0 0 0" xyz=" 0 0 0 "/>
+                <origin rpy="0 0 0" xyz=" 0 0 0 "/>
                 <geometry>
                     <mesh filename="package://reconcycle_description/meshes/tc_tool_side.obj" scale="0.001 0.001 0.001"/>

File: reconcycle_description/urdf/schunk_pzh20.xacro (robot description, xacro)
@@ -5,4 +5,40 @@
     </material>
     <xacro:arg name="schunk_gripper_id" default="schunk_pzh20"/>
+    <xacro:arg name="schunk_adapter_id" default="schunk_pzh20_adapter"/>
+     <link name="$(arg schunk_gripper_id)_base">
+    </link>
+    <joint name="griper_joint_base" type="fixed">
+        <parent link="$(arg schunk_gripper_id)_base"/>
+        <child link="$(arg schunk_adapter_id)"/>
+        <origin rpy="0 0 0" xyz="0 0 -0.02"/>
+    </joint>
+    <joint name="$griper_joint_adapter" type="fixed">
+        <parent link="$(arg schunk_adapter_id)"/>
+        <child link="$(arg schunk_gripper_id)"/>
+        <origin rpy="1.57 0 0" xyz="0 0 0"/>
+    </joint>
+    <material name="darkgray">
+    <color rgba="0.45 0.45 0.45 1"/>
+    </material>
+    <link name="$(arg schunk_adapter_id)">
+        <visual>
+            <origin rpy="0 0 0" xyz=" 0 0 0 "/>
+            <geometry>
+                <mesh filename="package://reconcycle_description/meshes/grippers/schunk_to_tc_adapter.stl" scale="0.001 0.001 0.001"/>
+            </geometry>
+            <material name="darkgray"/>
+        </visual>
+        <collision>
+            <origin rpy="0 0 0" xyz="0.0 0.0 0"/>
+            <geometry>
+                <mesh filename="package://reconcycle_description/meshes/grippers/schunk_to_tc_adapter.stl" scale ="0.001 0.001 0.001"/>
+            </geometry>
+        </collision>
+        <inertial>
+            <origin xyz="0 0 0" rpy="0 0 0"/>
+            <mass value="3"/>
+            <inertia ixx="3.0" ixy="0.0" ixz="0.0" iyy="3.0" iyz="0.0" izz="3.0"/>
+        </inertial>
+    </link>
     <link name="$(arg schunk_gripper_id)">
         <visual>
@@ -25,3 +61,5 @@
         </inertial>
     </link>
+    <xacro:include filename="$(find reconcycle_description)/urdf/reconcycle_defaults.xacro" />
+    <xacro:tc_tool_side tc_id="$(arg schunk_adapter_id)_tc_tool" connected_to="$(arg schunk_gripper_id)_base" xyz="0 0 -0.064" rpy='1.57 0 3.14'/>
 </robot>

File: reconcycle_description/urdf/tc_robot_side.xacro (robot description, xacro)
@@ -1,28 +1,15 @@
 <?xml version='1.0'?>
-<robot xmlns:xacro="http://www.ros.org/wiki/xacro" name="defaults">
-<xacro:macro name = "tc_robot" param="tc_id:='tc_robot' connected_to:='panda_link8'" >
-    <link name="${tc_id}">
+<robot xmlns:xacro="http://www.ros.org/wiki/xacro" name="tc_robot_side">
+    <xacro:arg name="base_link_name" default="tc_base_robot"/>
+    <xacro:arg name="robot_name" default="robot1"/>
+    <xacro:include filename="$(find reconcycle_description)/urdf/reconcycle_defaults.xacro" />
+    <link name="$(arg base_link_name)">
         <visual>
-            <origin rpy="1.57 0 -0.802664626" xyz=" 0 0 0 "/>
-            <geometry>
-                <mesh filename="package://reconcycle_description/meshes/tc_robot_side.obj" scale="0.001 0.001 0.001"/>
-            </geometry>
+                <origin rpy="0 0 0" xyz=" 0 0 -0.005 "/>
+                <geometry>
+                        <cylinder length="0.01" radius="0.03"/>
+                </geometry>
         </visual>
-        <collision>
-            <origin rpy="1.57 0 -0.802664626" xyz="0.0 0.0 0"/>
-            <geometry>
-                <mesh filename="package://reconcycle_description/meshes/tc_robot_side.obj" scale ="0.001 0.001 0.001"/>
-            </geometry>
-        </collision>
-        <inertial>
-            <origin xyz="0 0 0" rpy="0 0 0"/>
-            <mass value="3"/>
-            <inertia ixx="3.0" ixy="0.0" ixz="0.0" iyy="3.0" iyz="0.0" izz="3.0"/>
-        </inertial>
     </link>
-    <joint name="${tc_id}" type="fixed">
-        <parent link="${connected_to}"/>
-        <child link="${tc_id}"/>
-    </joint>
-</xacro:macro>
+    <xacro:tc_robot_side tc_id="$(arg robot_name)_tc_robot" connected_to="$(arg base_link_name)" xyz="0 0 0" rpy='0 0 0'/>
 </robot>
