Commit message: emo layout, modified vise obj

File: reconcycle_description/layouts/emo_layout.xacro (robot description, xacro)
@@ -3,6 +3,5 @@
     <link name="world"/>
     <!-- Usefull parameters -->
-    <!-- <xacro:include filename="$(find reconcycle_description)/urdf/reconcycle_defaults.xacro" /> -->
-    <xacro:include filename="$(find reconcycle_description)/urdf/reconcycle_default_models.xacro" />
+    <xacro:include filename="$(find reconcycle_description)/urdf/reconcycle_defaults.xacro" />
     <!-- Reconcycle table -->
     <xacro:include filename="$(find reconcycle_description)/urdf/table_module.xacro" />
@@ -10,22 +9,8 @@
     <xacro:arg name="table_0_name" default="table_rob_1"/>
     <xacro:arg name="table_1_name" default="table_cutting"/>
-    <xacro:arg name="table_2_name" default="table_tools"/>
     <xacro:arg name="table_3_name" default="table_fixture"/>
-    <!-- <xacro:arg name="table_4_name" default="table_output"/> -->
-    <xacro:arg name="table_5_name" default="table_rob_2"/>
-    <xacro:arg name="table_6_name" default="table_parts"/>
     <xacro:table_module table_id="$(arg table_0_name)" connected_to="world" xyz="0 0 ${table_height}" rpy="0 0 0"/>
     <xacro:table_module table_id="$(arg table_1_name)" connected_to="$(arg table_0_name)" xyz="0 -${table_width} 0" rpy="0 0 0"/>
-    <xacro:table_module table_id="$(arg table_2_name)" connected_to="$(arg table_0_name)" xyz="0 ${table_width} 0" rpy="0 0 0"/>
     <xacro:table_module table_id="$(arg table_3_name)" connected_to="$(arg table_0_name)" xyz="${table_width} 0 0" rpy="0 0 1.57"/>
-    <!-- <xacro:table_module table_id="$(arg table_4_name)" connected_to="$(arg table_3_name)" xyz="0 -${table_width} 0" rpy="0 0 0"/> -->
-    <xacro:table_module table_id="$(arg table_5_name)" connected_to="$(arg table_3_name)" xyz="${table_width} 0 0" rpy="0 0 3.14"/>
-    <xacro:table_module table_id="$(arg table_6_name)" connected_to="$(arg table_5_name)" xyz="0 ${table_width} 0" rpy="0 0 0"/>
-    <xacro:vise_setup_v2 connected_to="$(arg table_3_name)" xyz="0 0 0"/>
-    <xacro:cutter_model connected_to="$(arg table_6_name)" xyz="0 0 0" />
-    <xacro:tool_model connected_to="$(arg table_2_name)" xyz="0 0 0" />
-    <xacro:tool_frame_1 connected_to="$(arg table_2_name)" xyz="0.18 -0.036 0.355" rpy="0 3.1415 0" />
-    <xacro:tool_frame_2 connected_to="$(arg table_2_name)" xyz="0.06 -0.036 0.355" rpy="0 3.1415 0" />
-    <xacro:tool_frame_3 connected_to="$(arg table_2_name)" xyz="-0.06 -0.036 0.355" rpy="0 3.1415 0" />
-    <xacro:tool_frame_4 connected_to="$(arg table_2_name)" xyz="-0.18 -0.036 0.355" rpy="0 3.1415 0" />
+    <xacro:vise_setup connected_to="$(arg table_3_name)" xyz="0 0 0"/>
 </robot>

File: reconcycle_description/layouts/hca_layout.xacro (robot description, xacro)
@@ -3,6 +3,5 @@
     <link name="world"/>
     <!-- Usefull parameters -->
-    <!-- <xacro:include filename="$(find reconcycle_description)/urdf/reconcycle_defaults.xacro" /> -->
-    <xacro:include filename="$(find reconcycle_description)/urdf/reconcycle_default_models.xacro" />
+    <xacro:include filename="$(find reconcycle_description)/urdf/reconcycle_defaults.xacro" />
     <!-- Reconcycle table -->
     <xacro:include filename="$(find reconcycle_description)/urdf/table_module.xacro" />

File: reconcycle_description/urdf/panda_arm.xacro (robot description, xacro)
@@ -6,8 +6,8 @@
   <!-- <xacro:arg name="use_gazebo_control" default="false"/> -->
   <!-- <xacro:arg name="connected_to" default=""/> -->
-  <xacro:include filename="$(find franka_panda_description)/robots/panda_arm.xacro"/>
+  <xacro:include filename="$(find franka_description)/robots/panda_arm.xacro"/>
   <xacro:if value="${load_gazebo}">
-    <xacro:include filename="$(find franka_panda_description)/robots/panda.gazebo.xacro"/>
-    <xacro:include filename="$(find franka_panda_description)/robots/panda.transmission.xacro"/>
+    <xacro:include filename="$(find franka_description)/robots/panda.gazebo.xacro"/>
+    <xacro:include filename="$(find franka_description)/robots/panda.transmission.xacro"/>
     <xacro:panda_arm arm_id="${robot_name}" in_gazebo="true"  connected_to="${connected_to}"/>
     <xacro:panda_gazebo robot_name="${robot_name}" load_gripper="false"/>

File: reconcycle_description/urdf/reconcycle_defaults.xacro (robot description, xacro)
@@ -130,3 +130,220 @@
     </xacro:unless>
 </xacro:macro>
+<xacro:macro name="vise_setup_v2" params="vise_id:='vise' connected_to:='' xyz:='0 0 0' rpy='0 0 0'">
+    <!--  If connected_to is not provided we don't do anything -->
+    <xacro:unless value="${not connected_to}">
+        <joint name="${vise_id}_joint_${connected_to}" type="fixed">
+            <parent link="${connected_to}"/>
+            <child link="${vise_id}"/>
+            <origin rpy="${rpy}" xyz="${xyz}"/>
+            <dynamics damping="1"/>
+        </joint>
+        <!-- The vise -->
+        <link name="${vise_id}">
+            <visual>
+                <origin rpy="${pi/2} 0 0" xyz=" 0 0 0 "/>
+                <geometry>
+                    <mesh filename="package://reconcycle_description/meshes/vise_setup_v2.obj" scale="0.001 0.001 0.001"/>
+                </geometry>
+            </visual>
+            <collision>
+                <origin rpy="${pi/2} 0 0" xyz="0.0 0.0 0"/>
+                <geometry>
+                    <mesh filename="package://reconcycle_description/meshes/vise_setup_v2.obj" scale ="0.001 0.001 0.001"/>
+                </geometry>
+            </collision>
+            <inertial>
+                <origin xyz="0 0 0" rpy="0 0 0"/>
+                <mass value="3"/>
+                <inertia ixx="3.0" ixy="0.0" ixz="0.0" iyy="3.0" iyz="0.0" izz="3.0"/>
+            </inertial>
+        </link>
+    </xacro:unless>
+</xacro:macro>
+<xacro:macro name="cutter_model" params="cutter_id:='cutter' connected_to:='' xyz:='0 0 0' rpy='0 0 0'">
+    <!--  If connected_to is not provided we don't do anything -->
+    <xacro:unless value="${not connected_to}">
+        <joint name="${cutter_id}_joint_${connected_to}" type="fixed">
+            <parent link="${connected_to}"/>
+            <child link="${cutter_id}"/>
+            <origin rpy="${rpy}" xyz="${xyz}"/>
+            <dynamics damping="1"/>
+        </joint>
+        <!-- The vise -->
+        <link name="${cutter_id}">
+            <visual>
+                <origin rpy="${pi/2} 0 0" xyz=" 0 0 0 "/>
+                <geometry>
+                    <mesh filename="package://reconcycle_description/meshes/cutter_setup.obj" scale="0.001 0.001 0.001"/>
+                </geometry>
+            </visual>
+            <collision>
+                <origin rpy="${pi/2} 0 0" xyz="0.0 0.0 0"/>
+                <geometry>
+                    <mesh filename="package://reconcycle_description/meshes/cutter_setup.obj" scale ="0.001 0.001 0.001"/>
+                </geometry>
+            </collision>
+            <inertial>
+                <origin xyz="0 0 0" rpy="0 0 0"/>
+                <mass value="3"/>
+                <inertia ixx="3.0" ixy="0.0" ixz="0.0" iyy="3.0" iyz="0.0" izz="3.0"/>
+            </inertial>
+        </link>
+    </xacro:unless>
+</xacro:macro>
+<xacro:macro name="tool_model" params="tool_id:='tool' connected_to:='' xyz:='0 0 0' rpy='0 0 0'">
+    <!--  If connected_to is not provided we don't do anything -->
+    <xacro:unless value="${not connected_to}">
+        <joint name="${tool_id}_joint_${connected_to}" type="fixed">
+            <parent link="${connected_to}"/>
+            <child link="${tool_id}"/>
+            <origin rpy="${rpy}" xyz="${xyz}"/>
+            <dynamics damping="1"/>
+        </joint>
+        <!-- The vise -->
+        <link name="${tool_id}">
+            <visual>
+                <origin rpy="${pi/2} 0 0" xyz=" 0 0 0 "/>
+                <geometry>
+                    <mesh filename="package://reconcycle_description/meshes/toolholder_setup.obj" scale="0.001 0.001 0.001"/>
+                </geometry>
+            </visual>
+            <collision>
+                <origin rpy="${pi/2} 0 0" xyz="0.0 0.0 0"/>
+                <geometry>
+                    <mesh filename="package://reconcycle_description/meshes/toolholder_setup.obj" scale ="0.001 0.001 0.001"/>
+                </geometry>
+            </collision>
+            <inertial>
+                <origin xyz="0 0 0" rpy="0 0 0"/>
+                <mass value="3"/>
+                <inertia ixx="3.0" ixy="0.0" ixz="0.0" iyy="3.0" iyz="0.0" izz="3.0"/>
+            </inertial>
+        </link>
+    </xacro:unless>
+</xacro:macro>
+<xacro:macro name="tool_frame_1" params="tool_id:='tool_frame_1' connected_to:='' xyz:='0.0 0.0 0.0' rpy='0 0 0'">
+    <!--  If connected_to is not provided we don't do anything -->
+    <xacro:unless value="${not connected_to}">
+        <joint name="${tool_id}_joint_${connected_to}" type="fixed">
+            <parent link="${connected_to}"/>
+            <child link="${tool_id}"/>
+            <origin rpy="${rpy}" xyz="${xyz}"/>
+            <dynamics damping="1"/>
+        </joint>
+        <!-- The vise -->
+        <link name="${tool_id}">
+            <visual>
+                <origin rpy="${pi/2} 0 0" xyz=" 0 0 0 "/>
+                <geometry>
+                    <mesh filename="package://reconcycle_description/meshes/EmptyCubeFrame.obj" scale="0.001 0.001 0.001"/>
+                </geometry>
+            </visual>
+            <collision>
+                <origin rpy="${pi/2} 0 0" xyz="0.0 0.0 0"/>
+                <geometry>
+                    <mesh filename="package://reconcycle_description/meshes/EmptyCubeFrame.obj" scale ="0.001 0.001 0.001"/>
+                </geometry>
+            </collision>
+            <inertial>
+                <origin xyz="0 0 0" rpy="0 0 0"/>
+                <mass value="3"/>
+                <inertia ixx="3.0" ixy="0.0" ixz="0.0" iyy="3.0" iyz="0.0" izz="3.0"/>
+            </inertial>
+        </link>
+    </xacro:unless>
+</xacro:macro>
+<xacro:macro name="tool_frame_2" params="tool_id:='tool_frame_2' connected_to:='' xyz:='0.0 0.0 0.0' rpy='0 0 0'">
+    <!--  If connected_to is not provided we don't do anything -->
+    <xacro:unless value="${not connected_to}">
+        <joint name="${tool_id}_joint_${connected_to}" type="fixed">
+            <parent link="${connected_to}"/>
+            <child link="${tool_id}"/>
+            <origin rpy="${rpy}" xyz="${xyz}"/>
+            <dynamics damping="1"/>
+        </joint>
+        <!-- The vise -->
+        <link name="${tool_id}">
+            <visual>
+                <origin rpy="${pi/2} 0 0" xyz=" 0 0 0 "/>
+                <geometry>
+                    <mesh filename="package://reconcycle_description/meshes/EmptyCubeFrame.obj" scale="0.001 0.001 0.001"/>
+                </geometry>
+            </visual>
+            <collision>
+                <origin rpy="${pi/2} 0 0" xyz="0.0 0.0 0"/>
+                <geometry>
+                    <mesh filename="package://reconcycle_description/meshes/EmptyCubeFrame.obj" scale ="0.001 0.001 0.001"/>
+                </geometry>
+            </collision>
+            <inertial>
+                <origin xyz="0 0 0" rpy="0 0 0"/>
+                <mass value="3"/>
+                <inertia ixx="3.0" ixy="0.0" ixz="0.0" iyy="3.0" iyz="0.0" izz="3.0"/>
+            </inertial>
+        </link>
+    </xacro:unless>
+</xacro:macro>
+<xacro:macro name="tool_frame_3" params="tool_id:='tool_frame_3' connected_to:='' xyz:='0.0 0.0 0.0' rpy='0 0 0'">
+    <!--  If connected_to is not provided we don't do anything -->
+    <xacro:unless value="${not connected_to}">
+        <joint name="${tool_id}_joint_${connected_to}" type="fixed">
+            <parent link="${connected_to}"/>
+            <child link="${tool_id}"/>
+            <origin rpy="${rpy}" xyz="${xyz}"/>
+            <dynamics damping="1"/>
+        </joint>
+        <!-- The vise -->
+        <link name="${tool_id}">
+            <visual>
+                <origin rpy="${pi/2} 0 0" xyz=" 0 0 0 "/>
+                <geometry>
+                    <mesh filename="package://reconcycle_description/meshes/EmptyCubeFrame.obj" scale="0.001 0.001 0.001"/>
+                </geometry>
+            </visual>
+            <collision>
+                <origin rpy="${pi/2} 0 0" xyz="0.0 0.0 0"/>
+                <geometry>
+                    <mesh filename="package://reconcycle_description/meshes/EmptyCubeFrame.obj" scale ="0.001 0.001 0.001"/>
+                </geometry>
+            </collision>
+            <inertial>
+                <origin xyz="0 0 0" rpy="0 0 0"/>
+                <mass value="3"/>
+                <inertia ixx="3.0" ixy="0.0" ixz="0.0" iyy="3.0" iyz="0.0" izz="3.0"/>
+            </inertial>
+        </link>
+    </xacro:unless>
+</xacro:macro>
+<xacro:macro name="tool_frame_4" params="tool_id:='tool_frame_4' connected_to:='' xyz:='0.0 0.0 0.0' rpy='0 0 0'">
+    <!--  If connected_to is not provided we don't do anything -->
+    <xacro:unless value="${not connected_to}">
+        <joint name="${tool_id}_joint_${connected_to}" type="fixed">
+            <parent link="${connected_to}"/>
+            <child link="${tool_id}"/>
+            <origin rpy="${rpy}" xyz="${xyz}"/>
+            <dynamics damping="1"/>
+        </joint>
+        <!-- The vise -->
+        <link name="${tool_id}">
+            <visual>
+                <origin rpy="${pi/2} 0 0" xyz=" 0 0 0 "/>
+                <geometry>
+                    <mesh filename="package://reconcycle_description/meshes/EmptyCubeFrame.obj" scale="0.001 0.001 0.001"/>
+                </geometry>
+            </visual>
+            <collision>
+                <origin rpy="${pi/2} 0 0" xyz="0.0 0.0 0"/>
+                <geometry>
+                    <mesh filename="package://reconcycle_description/meshes/EmptyCubeFrame.obj" scale ="0.001 0.001 0.001"/>
+                </geometry>
+            </collision>
+            <inertial>
+                <origin xyz="0 0 0" rpy="0 0 0"/>
+                <mass value="3"/>
+                <inertia ixx="3.0" ixy="0.0" ixz="0.0" iyy="3.0" iyz="0.0" izz="3.0"/>
+            </inertial>
+        </link>
+    </xacro:unless>
+</xacro:macro>
 </robot>

File: reconcycle_description/urdf/reconcycle_panda.xacro (robot description, xacro)
@@ -7,11 +7,14 @@
     <xacro:include filename="$(find reconcycle_description)/urdf/reconcycle_defaults.xacro" />
     <!-- Load the reconcycle panda macro  -->
-    <xacro:include filename="$(find reconcycle_description)/urdf/panda_arm.xacro"/>
-    <!-- Create a default world link but it's not called world -->
-    <link name="$(arg robot_name)" />
+    <!--<xacro:include filename="$(find reconcycle_description)/urdf/panda_arm.xacro"/> -->
+    <xacro:include filename="$(find franka_description)/robots/panda_arm.xacro"/>
+    <!-- Create a default world link but it's not called world
+    <link name="$(arg robot_name)" />-->
     <!-- Call the macro -->
-    <xacro:panda_robot load_gazebo="$(arg load_gazebo)" robot_name="$(arg robot_name)" connected_to="$(arg robot_name)"/>
-    <!-- Attach the flange to the robot -->
-    <xacro:flange flange_id="$(arg robot_name)_flange" connected_to="$(arg robot_name)_link8"/>
+    <!--<xacro:panda_robot load_gazebo="$(arg load_gazebo)" robot_name="$(arg robot_name)" connected_to="$(arg robot_name)"/> -->
+    <xacro:panda_arm arm_id="$(arg robot_name)" connected_to="$(arg connected_to)"/>
+    <!-- Attach the flange to the robot
+    <xacro:flange flange_id="$(arg robot_name)_flange" connected_to="$(arg robot_name)_link8"/>-->
+    <xacro:flange flange_id="panda_flange" connected_to="panda_link8"/>
     <!-- Attach the tool exchange to the robot -->
     <xacro:tc_robot_side tc_id="$(arg robot_name)_tc_robot" connected_to="$(arg robot_name)_flange" xyz="0 0 ${flange_thickness}"/>
