Commit message: upd

File: reconcycle_description/layouts/qundis_layout.xacro (robot description, xacro)
@@ -2,5 +2,5 @@
 <robot xmlns:xacro="http://www.ros.org/wiki/xacro" name="reconcycle" >
     <link name="world"/>
-    <!-- Usefull parameters -->
+    <!-- Useful parameters -->
     <xacro:include filename="$(find reconcycle_description)/urdf/reconcycle_defaults.xacro" />
     <!-- Reconcycle table -->
@@ -10,12 +10,12 @@
     <xacro:arg name="table_1_name" default="table_vision"/>
     <xacro:arg name="table_2_name" default="table_fixture"/>
-    <xacro:arg name="table_3_name" default="table_rob_2"/>
-    <xacro:arg name="table_4_name" default="table_cutter"/>
+    <xacro:arg name="table_3_name" default="table_cutter"/>
+    <xacro:arg name="table_4_name" default="table_rob_2"/>
     <xacro:table_module table_id="$(arg table_0_name)" connected_to="world" xyz="0 0 ${table_height}" rpy="0 0 0"/>
     <xacro:table_module table_id="$(arg table_1_name)" connected_to="$(arg table_0_name)" xyz="${table_width} 0 0" rpy="0 0 0"/>
     <xacro:table_module table_id="$(arg table_2_name)" connected_to="$(arg table_0_name)" xyz="${table_width} -${table_width} 0" rpy="0 0 1.57"/>
     <xacro:table_module table_id="$(arg table_3_name)" connected_to="$(arg table_1_name)" xyz="${table_width} 0 0" rpy="0 0 0"/>
-    <xacro:table_module table_id="$(arg table_4_name)" connected_to="$(arg table_1_name)" xyz="${table_width} -${table_width} 0" rpy="0 0 -3.14"/>
+    <xacro:table_module table_id="$(arg table_4_name)" connected_to="$(arg table_1_name)" xyz="${table_width} -${table_width} 0" rpy="0 0 0"/>
     <xacro:vise_setup connected_to="$(arg table_2_name)" xyz="0 0 0"/>
-    <xacro:cutter_model connected_to="$(arg table_4_name)" xyz="0 0 0"/>
+    <xacro:cutter_model connected_to="$(arg table_3_name)" xyz="0 0 0" rpy="0 0 -1.5708"/>
 </robot>

File: reconcycle_description/urdf/screwdriver.xacro (robot description, xacro)
@@ -1,5 +1,6 @@
 <?xml version='1.0'?>
 <robot xmlns:xacro="http://www.ros.org/wiki/xacro" name="defaults">
-    <link name="screwdriver">
+    <xacro:arg name="screwdriver_id" default="screwdriver_panda_2"/>
+    <link name="$(arg screwdriver_id">
         <visual>
             <origin rpy="1.57 0 0" xyz=" 0 0 0 "/>
