Commit message: add robotic_cell_description, add schunk 3jaw urdf, add cnc model

File: reconcycle_module_cnc/urdf/reconcycle_module_cnc.urdf (robot description, URDF)
Before this commit: robot fifi, 13 links, 12 joints
Links:
- added link clamp1
- added link clamp2
- added link cnctable
- link base: geometry visual mesh filename=package://reconcycle_module_cnc/meshes/095-000-002-DIN63210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; visual mesh filename=package://reconcycle_module_cnc/meshes/095-000-002-DIN63211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
Joints:
- removed joint base_cncbase
- added joint base_cnctable: type fixed, parent base, child cnctable, origin xyz=0.3000000000000018 0.3000000000000216 1.9554136088117956e-14 rpy=2.2579430955137512e-28 -2.508342171493172e-16 1.1143863609679275e-14, axis 1 0 0, limit lower=-1.548 upper=1.548 effort=1000 velocity=0.5
- added joint cncbase_clamp1: type fixed, parent cncbase, child clamp1, origin xyz=-0.04900000000000071 -0.15400000000002348 -0.10000000000000592 rpy=-2.1960919458032578e-16 3.4759354975015094e-14 -1.5707963267949014, axis 1 0 0, limit lower=-1.548 upper=1.548 effort=1000 velocity=0.5
- added joint cncbase_clamp2: type fixed, parent cncbase, child clamp2, origin xyz=-0.31000000000013944 -0.15400000000000033 -0.09763116166886766 rpy=1.4477308241114202e-13 -5.551115124530586e-17 -1.5707963267949014, axis 1 0 0, limit lower=-1.548 upper=1.548 effort=1000 velocity=0.5
- added joint cnctable_cncbase: type fixed, parent cnctable, child cncbase, origin xyz=-0.09000000000002663 0.18999999999997152 0.10000000000000682 rpy=-3.474791259756282e-14 -3.5103864259878375e-14 1.5707963267949014, axis 1 0 0, limit lower=-1.548 upper=1.548 effort=1000 velocity=0.5
- joint cncbase_xAxis: origin xyz=-1.0913936421275139e-14 0.0 1.0118128557223826e-14 rpy=3.1337803125299106 1.5707963267948877 3.133780312529911 -> xyz=1.1368683772161603e-15 -1.4766499134566402e-13 -5.115907697472721e-15 rpy=3.5971469538897717e-13 4.392183891463523e-16 1.6209639865544653e-15
- joint xAxis_yAxis: origin xyz=0.2400000000000092 -8.242295734817162e-15 0.20000000000000973 rpy=-1.5707963267948923 8.327642916791075e-17 7.354144300786629e-16 -> xyz=-1.1937117960769684e-15 1.4772183476452482e-13 4.888534022029489e-15 rpy=-8.93715939841262e-16 3.597146953889761e-13 1.5707963267949
- joint yAxis_zAxis: origin xyz=8.86757334228605e-15 -0.16500000000000134 0.2800000000000127 rpy=3.0999500744925093 -1.5707963267948766 -3.0999500744925097 -> xyz=-4.4622083805734293e-14 -9.663381206337363e-16 4.547473508864641e-16 rpy=-3.0256378814571314 -1.5707963267948917 3.02563788145711
