Commit message: add robotic_cell_description, add schunk 3jaw urdf, add cnc model

File: reconcycle_module_cnc/urdf/reconcycle_module_cnc.urdf.xacro (robot description, xacro)
@@ -3,8 +3,11 @@
 <xacro:macro name="my_robot" params="robot_name">
 <xacro:property name="robot_prefix" value="${robot_name}" />
+<xacro:property name="joint_14_name" value="${robot_prefix}base_cnctable" />
+<xacro:property name="joint_13_name" value="${robot_prefix}cncbase_clamp2" />
+<xacro:property name="joint_12_name" value="${robot_prefix}cncbase_clamp1" />
 <xacro:property name="joint_11_name" value="${robot_prefix}yAxis_zAxis" />
 <xacro:property name="joint_10_name" value="${robot_prefix}xAxis_yAxis" />
 <xacro:property name="joint_9_name" value="${robot_prefix}cncbase_xAxis" />
-<xacro:property name="joint_8_name" value="${robot_prefix}base_cncbase" />
+<xacro:property name="joint_8_name" value="${robot_prefix}cnctable_cncbase" />
 <xacro:property name="joint_7_name" value="${robot_prefix}base_pnpf4" />
 <xacro:property name="joint_6_name" value="${robot_prefix}base_pnpf" />
@@ -15,7 +18,10 @@
 <xacro:property name="joint_1_name" value="${robot_prefix}base_pnpm1" />
 <xacro:property name="joint_0_name" value="${robot_prefix}base_pnpm2" />
-<xacro:property name="link_12_name" value="${robot_prefix}zAxis" />
-<xacro:property name="link_11_name" value="${robot_prefix}yAxis" />
-<xacro:property name="link_10_name" value="${robot_prefix}xAxis" />
+<xacro:property name="link_15_name" value="${robot_prefix}clamp2" />
+<xacro:property name="link_14_name" value="${robot_prefix}clamp1" />
+<xacro:property name="link_13_name" value="${robot_prefix}zAxis" />
+<xacro:property name="link_12_name" value="${robot_prefix}yAxis" />
+<xacro:property name="link_11_name" value="${robot_prefix}xAxis" />
+<xacro:property name="link_10_name" value="${robot_prefix}cnctable" />
 <xacro:property name="link_9_name" value="${robot_prefix}cncbase" />
 <xacro:property name="link_8_name" value="${robot_prefix}pnpf4" />
@@ -85,26 +91,19 @@
   </joint>
   <joint name="${joint_8_name}" type="fixed">
-    <origin xyz="0.049999999999967 0.5750000000000004 0.09999999999788053" rpy="-3.141592653589689 -4.957596153306171e-14 1.2476131239222398e-14"/>
+    <origin xyz="-0.09000000000002663 0.18999999999997152 0.10000000000000682" rpy="-3.474791259756282e-14 -3.5103864259878375e-14 1.5707963267949014"/>
     <axis xyz="1 0 0"/>
-    <parent link="${link_1_name}"/>
+    <parent link="${link_10_name}"/>
     <child link="${link_9_name}"/>
     <limit effort="1000" lower="-1.548" upper="1.548" velocity="0.5"/>
   </joint>
   <joint name="${joint_9_name}" type="prismatic">
-    <origin xyz="-1.0913936421275139e-14 0.0 1.0118128557223826e-14" rpy="3.1337803125299106 1.5707963267948877 3.133780312529911"/>
+    <origin xyz="1.1368683772161603e-15 -1.4766499134566402e-13 -5.115907697472721e-15" rpy="3.5971469538897717e-13 4.392183891463523e-16 1.6209639865544653e-15"/>
     <axis xyz="1 0 0"/>
     <parent link="${link_9_name}"/>
-    <child link="${link_10_name}"/>
+    <child link="${link_11_name}"/>
     <limit effort="1000" lower="-1.548" upper="1.548" velocity="0.5"/>
   </joint>
   <joint name="${joint_10_name}" type="prismatic">
-    <origin xyz="0.2400000000000092 -8.242295734817162e-15 0.20000000000000973" rpy="-1.5707963267948923 8.327642916791075e-17 7.354144300786629e-16"/>
-    <axis xyz="1 0 0"/>
-    <parent link="${link_10_name}"/>
-    <child link="${link_11_name}"/>
-    <limit effort="1000" lower="-1.548" upper="1.548" velocity="0.5"/>
-  </joint>
-  <joint name="${joint_11_name}" type="prismatic">
-    <origin xyz="8.86757334228605e-15 -0.16500000000000134 0.2800000000000127" rpy="3.0999500744925093 -1.5707963267948766 -3.0999500744925097"/>
+    <origin xyz="-1.1937117960769684e-15 1.4772183476452482e-13 4.888534022029489e-15" rpy="-8.93715939841262e-16 3.597146953889761e-13 1.5707963267949"/>
     <axis xyz="1 0 0"/>
     <parent link="${link_11_name}"/>
@@ -112,4 +111,32 @@
     <limit effort="1000" lower="-1.548" upper="1.548" velocity="0.5"/>
   </joint>
+  <joint name="${joint_11_name}" type="prismatic">
+    <origin xyz="-4.4622083805734293e-14 -9.663381206337363e-16 4.547473508864641e-16" rpy="-3.0256378814571314 -1.5707963267948917 3.02563788145711"/>
+    <axis xyz="1 0 0"/>
+    <parent link="${link_12_name}"/>
+    <child link="${link_13_name}"/>
+    <limit effort="1000" lower="-1.548" upper="1.548" velocity="0.5"/>
+  </joint>
+  <joint name="${joint_12_name}" type="fixed">
+    <origin xyz="-0.04900000000000071 -0.15400000000002348 -0.10000000000000592" rpy="-2.1960919458032578e-16 3.4759354975015094e-14 -1.5707963267949014"/>
+    <axis xyz="1 0 0"/>
+    <parent link="${link_9_name}"/>
+    <child link="${link_14_name}"/>
+    <limit effort="1000" lower="-1.548" upper="1.548" velocity="0.5"/>
+  </joint>
+  <joint name="${joint_13_name}" type="fixed">
+    <origin xyz="-0.31000000000013944 -0.15400000000000033 -0.09763116166886766" rpy="1.4477308241114202e-13 -5.551115124530586e-17 -1.5707963267949014"/>
+    <axis xyz="1 0 0"/>
+    <parent link="${link_9_name}"/>
+    <child link="${link_15_name}"/>
+    <limit effort="1000" lower="-1.548" upper="1.548" velocity="0.5"/>
+  </joint>
+  <joint name="${joint_14_name}" type="fixed">
+    <origin xyz="0.3000000000000018 0.3000000000000216 1.9554136088117956e-14" rpy="2.2579430955137512e-28 -2.508342171493172e-16 1.1143863609679275e-14"/>
+    <axis xyz="1 0 0"/>
+    <parent link="${link_1_name}"/>
+    <child link="${link_10_name}"/>
+    <limit effort="1000" lower="-1.548" upper="1.548" velocity="0.5"/>
+  </joint>
   <link name="${link_0_name}"/>
   <link name="${link_1_name}">
@@ -3024,2336 +3051,356 @@
       <origin xyz="0.30000000000004 0.30000000000003446 -0.9065740663179903" rpy="2.1563646842988024e-14 3.504835310863548e-14 -1.5707963267948966"/>
       <geometry>
-        <mesh filename="package://reconcycle_module_cnc/meshes/PENN_ELCOM-R1290-1U_R1290-91_BR0.stl"/>
+        <mesh filename="package://reconcycle_module_cnc/meshes/HRP-POA_50G_7570190.stl"/>
+      </geometry>
+      <material name="color2">
+        <color rgba="0.35153260827064514 0.35153260827064514 0.35153260827064514 1"/>
+      </material>
+    </visual>
+    <visual>
+      <origin xyz="0.30000000000004 0.30000000000003446 -0.9065740663179903" rpy="2.1563646842988024e-14 3.504835310863548e-14 -1.5707963267948966"/>
+      <geometry>
+        <mesh filename="package://reconcycle_module_cnc/meshes/HRP-POA_50G_7570191.stl"/>
+      </geometry>
+      <material name="color2">
+        <color rgba="0.35153260827064514 0.35153260827064514 0.35153260827064514 1"/>
+      </material>
+    </visual>
+    <visual>
+      <origin xyz="0.30000000000004 0.30000000000003446 -0.9065740663179903" rpy="2.1563646842988024e-14 3.504835310863548e-14 -1.5707963267948966"/>
+      <geometry>
+        <mesh filename="package://reconcycle_module_cnc/meshes/HRP-POA_50G_7570192.stl"/>
+      </geometry>
+      <material name="color2">
+        <color rgba="0.35153260827064514 0.35153260827064514 0.35153260827064514 1"/>
+      </material>
+    </visual>
+    <visual>
+      <origin xyz="0.30000000000004 0.30000000000003446 -0.9065740663179903" rpy="2.1563646842988024e-14 3.504835310863548e-14 -1.5707963267948966"/>
+      <geometry>
+        <mesh filename="package://reconcycle_module_cnc/meshes/HRP-POA_50G_7570193.stl"/>
+      </geometry>
+      <material name="color2">
+        <color rgba="0.35153260827064514 0.35153260827064514 0.35153260827064514 1"/>
+      </material>
+    </visual>
+    <visual>
+      <origin xyz="0.30000000000004 0.30000000000003446 -0.9065740663179903" rpy="2.1563646842988024e-14 3.504835310863548e-14 -1.5707963267948966"/>
+      <geometry>
+        <mesh filename="package://reconcycle_module_cnc/meshes/RCY-099-005-0010.stl"/>
+      </geometry>
+      <material name="color2">
+        <color rgba="0.35153260827064514 0.35153260827064514 0.35153260827064514 1"/>
+      </material>
+    </visual>
+    <visual>
+      <origin xyz="0.30000000000004 0.30000000000003446 -0.9065740663179903" rpy="2.1563646842988024e-14 3.504835310863548e-14 -1.5707963267948966"/>
+      <geometry>
+        <mesh filename="package://reconcycle_module_cnc/meshes/RCY-099-005-0011.stl"/>
+      </geometry>
+      <material name="color2">
+        <color rgba="0.35153260827064514 0.35153260827064514 0.35153260827064514 1"/>
+      </material>
+    </visual>
+    <visual>
+      <origin xyz="0.30000000000004 0.30000000000003446 -0.9065740663179903" rpy="2.1563646842988024e-14 3.504835310863548e-14 -1.5707963267948966"/>
+      <geometry>
+        <mesh filename="package://reconcycle_module_cnc/meshes/RCY-099-005-0012.stl"/>
+      </geometry>
+      <material name="color2">
+        <color rgba="0.35153260827064514 0.35153260827064514 0.35153260827064514 1"/>
+      </material>
+    </visual>
+    <visual>
+      <origin xyz="0.30000000000004 0.30000000000003446 -0.9065740663179903" rpy="2.1563646842988024e-14 3.504835310863548e-14 -1.5707963267948966"/>
+      <geometry>
+        <mesh filename="package://reconcycle_module_cnc/meshes/RCY-099-005-0013.stl"/>
+      </geometry>
+      <material name="color2">
+        <color rgba="0.35153260827064514 0.35153260827064514 0.35153260827064514 1"/>
+      </material>
+    </visual>
+    <visual>
+      <origin xyz="0.30000000000004 0.30000000000003446 -0.9065740663179903" rpy="2.1563646842988024e-14 3.504835310863548e-14 -1.5707963267948966"/>
+      <geometry>
+        <mesh filename="package://reconcycle_module_cnc/meshes/SIDE_BEAM0.stl"/>
+      </geometry>
+      <material name="color2">
+        <color rgba="0.35153260827064514 0.35153260827064514 0.35153260827064514 1"/>
+      </material>
+    </visual>
+    <visual>
+      <origin xyz="0.30000000000004 0.30000000000003446 -0.9065740663179903" rpy="2.1563646842988024e-14 3.504835310863548e-14 -1.5707963267948966"/>
+      <geometry>
+        <mesh filename="package://reconcycle_module_cnc/meshes/FRONT_BEAM0.stl"/>
+      </geometry>
+      <material name="color2">
+        <color rgba="0.35153260827064514 0.35153260827064514 0.35153260827064514 1"/>
+      </material>
+    </visual>
+    <visual>
+      <origin xyz="0.30000000000004 0.30000000000003446 -0.9065740663179903" rpy="2.1563646842988024e-14 3.504835310863548e-14 -1.5707963267948966"/>
+      <geometry>
+        <mesh filename="package://reconcycle_module_cnc/meshes/FRONT_BEAM1.stl"/>
+      </geometry>
+      <material name="color2">
+        <color rgba="0.35153260827064514 0.35153260827064514 0.35153260827064514 1"/>
+      </material>
+    </visual>
+    <visual>
+      <origin xyz="0.30000000000004 0.30000000000003446 -0.9065740663179903" rpy="2.1563646842988024e-14 3.504835310863548e-14 -1.5707963267948966"/>
+      <geometry>
+        <mesh filename="package://reconcycle_module_cnc/meshes/SIDE_BEAM1.stl"/>
+      </geometry>
+      <material name="color2">
+        <color rgba="0.35153260827064514 0.35153260827064514 0.35153260827064514 1"/>
+      </material>
+    </visual>
+    <visual>
+      <origin xyz="0.30000000000004 0.30000000000003446 -0.9065740663179903" rpy="2.1563646842988024e-14 3.504835310863548e-14 -1.5707963267948966"/>
+      <geometry>
+        <mesh filename="package://reconcycle_module_cnc/meshes/SIDE_BRACKET0.stl"/>
+      </geometry>
+      <material name="color2">
+        <color rgba="0.35153260827064514 0.35153260827064514 0.35153260827064514 1"/>
+      </material>
+    </visual>
+    <visual>
+      <origin xyz="0.30000000000004 0.30000000000003446 -0.9065740663179903" rpy="2.1563646842988024e-14 3.504835310863548e-14 -1.5707963267948966"/>
+      <geometry>
+        <mesh filename="package://reconcycle_module_cnc/meshes/SIDE_BRACKET1.stl"/>
+      </geometry>
+      <material name="color2">
+        <color rgba="0.35153260827064514 0.35153260827064514 0.35153260827064514 1"/>
+      </material>
+    </visual>
+    <visual>
+      <origin xyz="0.30000000000004 0.30000000000003446 -0.9065740663179903" rpy="2.1563646842988024e-14 3.504835310863548e-14 -1.5707963267948966"/>
+      <geometry>
+        <mesh filename="package://reconcycle_module_cnc/meshes/SIDE_BRACKET2.stl"/>
+      </geometry>
+      <material name="color2">
+        <color rgba="0.35153260827064514 0.35153260827064514 0.35153260827064514 1"/>
+      </material>
+    </visual>
+    <visual>
+      <origin xyz="0.30000000000004 0.30000000000003446 -0.9065740663179903" rpy="2.1563646842988024e-14 3.504835310863548e-14 -1.5707963267948966"/>
+      <geometry>
+        <mesh filename="package://reconcycle_module_cnc/meshes/SIDE_BRACKET3.stl"/>
+      </geometry>
+      <material name="color2">
+        <color rgba="0.35153260827064514 0.35153260827064514 0.35153260827064514 1"/>
+      </material>
+    </visual>
+    <visual>
+      <origin xyz="0.30000000000004 0.30000000000003446 -0.9065740663179903" rpy="2.1563646842988024e-14 3.504835310863548e-14 -1.5707963267948966"/>
+      <geometry>
+        <mesh filename="package://reconcycle_module_cnc/meshes/MOTOR0.stl"/>
+      </geometry>
+      <material name="color2">
+        <color rgba="0.35153260827064514 0.35153260827064514 0.35153260827064514 1"/>
+      </material>
+    </visual>
+    <visual>
+      <origin xyz="0.30000000000004 0.30000000000003446 -0.9065740663179903" rpy="2.1563646842988024e-14 3.504835310863548e-14 -1.5707963267948966"/>
+      <geometry>
+        <mesh filename="package://reconcycle_module_cnc/meshes/MOTOR1.stl"/>
+      </geometry>
+      <material name="color2">
+        <color rgba="0.35153260827064514 0.35153260827064514 0.35153260827064514 1"/>
+      </material>
+    </visual>
+    <visual>
+      <origin xyz="0.30000000000004 0.30000000000003446 -0.9065740663179903" rpy="2.1563646842988024e-14 3.504835310863548e-14 -1.5707963267948966"/>
+      <geometry>
+        <mesh filename="package://reconcycle_module_cnc/meshes/SCHUNK-5517153-Gehaeuse-JGZ-800.stl"/>
       </geometry>
       <material name="color9">
-        <color rgba="0.5906188488006592 0.637596845626831 0.8549926280975342 1"/>
-      </material>
-    </visual>
-    <visual>
-      <origin xyz="0.30000000000004 0.30000000000003446 -0.9065740663179903" rpy="2.1563646842988024e-14 3.504835310863548e-14 -1.5707963267948966"/>
-      <geometry>
-        <mesh filename="package://reconcycle_module_cnc/meshes/PENN_ELCOM-R1290-1U_R1290-1U_TR0.stl"/>
+        <color rgba="0.3049873113632202 0.3049873113632202 0.07036009430885315 1"/>
+      </material>
+    </visual>
+    <visual>
+      <origin xyz="0.30000000000004 0.30000000000003446 -0.9065740663179903" rpy="2.1563646842988024e-14 3.504835310863548e-14 -1.5707963267948966"/>
+      <geometry>
+        <mesh filename="package://reconcycle_module_cnc/meshes/SCHUNK-5503506-Halter-fuer-NHS-KL030.stl"/>
+      </geometry>
+      <material name="color2">
+        <color rgba="0.35153260827064514 0.35153260827064514 0.35153260827064514 1"/>
+      </material>
+    </visual>
+    <visual>
+      <origin xyz="0.30000000000004 0.30000000000003446 -0.9065740663179903" rpy="2.1563646842988024e-14 3.504835310863548e-14 -1.5707963267948966"/>
+      <geometry>
+        <mesh filename="package://reconcycle_module_cnc/meshes/SCHUNK-5503506-Halter-fuer-NHS-KL031.stl"/>
+      </geometry>
+      <material name="color2">
+        <color rgba="0.35153260827064514 0.35153260827064514 0.35153260827064514 1"/>
+      </material>
+    </visual>
+    <visual>
+      <origin xyz="0.30000000000004 0.30000000000003446 -0.9065740663179903" rpy="2.1563646842988024e-14 3.504835310863548e-14 -1.5707963267948966"/>
+      <geometry>
+        <mesh filename="package://reconcycle_module_cnc/meshes/SCHUNK-5503506-Halter-fuer-NHS-KL032.stl"/>
+      </geometry>
+      <material name="color2">
+        <color rgba="0.35153260827064514 0.35153260827064514 0.35153260827064514 1"/>
+      </material>
+    </visual>
+    <visual>
+      <origin xyz="0.30000000000004 0.30000000000003446 -0.9065740663179903" rpy="2.1563646842988024e-14 3.504835310863548e-14 -1.5707963267948966"/>
+      <geometry>
+        <mesh filename="package://reconcycle_module_cnc/meshes/SCHUNK-Cover-JGZ-800.stl"/>
+      </geometry>
+      <material name="color2">
+        <color rgba="0.35153260827064514 0.35153260827064514 0.35153260827064514 1"/>
+      </material>
+    </visual>
+    <visual>
+      <origin xyz="0.30000000000004 0.30000000000003446 -0.9065740663179903" rpy="2.1563646842988024e-14 3.504835310863548e-14 -1.5707963267948966"/>
+      <geometry>
+        <mesh filename="package://reconcycle_module_cnc/meshes/SCHUNK-9905500-Typenschild-5x20x0.30.stl"/>
+      </geometry>
+      <material name="color2">
+        <color rgba="0.35153260827064514 0.35153260827064514 0.35153260827064514 1"/>
+      </material>
+    </visual>
+    <visual>
+      <origin xyz="0.30000000000004 0.30000000000003446 -0.9065740663179903" rpy="2.1563646842988024e-14 3.504835310863548e-14 -1.5707963267948966"/>
+      <geometry>
+        <mesh filename="package://reconcycle_module_cnc/meshes/SCHUNK-5512155-Deckel-PZN+80_JGZ80_DPZ+800.stl"/>
       </geometry>
       <material name="color10">
-        <color rgba="0.009721217676997185 0.009721217676997185 0.009721217676997185 1"/>
-      </material>
-    </visual>
-    <visual>
-      <origin xyz="0.30000000000004 0.30000000000003446 -0.9065740663179903" rpy="2.1563646842988024e-14 3.504835310863548e-14 -1.5707963267948966"/>
-      <geometry>
-        <mesh filename="package://reconcycle_module_cnc/meshes/PENN_ELCOM-R1290-1U_R1290-91_BR1.stl"/>
+        <color rgba="0.35153260827064514 0.35153260827064514 0.0802198201417923 1"/>
+      </material>
+    </visual>
+    <visual>
+      <origin xyz="0.30000000000004 0.30000000000003446 -0.9065740663179903" rpy="2.1563646842988024e-14 3.504835310863548e-14 -1.5707963267948966"/>
+      <geometry>
+        <mesh filename="package://reconcycle_module_cnc/meshes/SCHUNK-5517091-finger-JGP-80-1-_-JGZ-80-10.stl"/>
+      </geometry>
+      <material name="color11">
+        <color rgba="0.023153366521000862 0.023153366521000862 0.023153366521000862 1"/>
+      </material>
+    </visual>
+    <visual>
+      <origin xyz="0.30000000000004 0.30000000000003446 -0.9065740663179903" rpy="2.1563646842988024e-14 3.504835310863548e-14 -1.5707963267948966"/>
+      <geometry>
+        <mesh filename="package://reconcycle_module_cnc/meshes/SCHUNK-5517091-finger-JGP-80-1-_-JGZ-80-11.stl"/>
+      </geometry>
+      <material name="color11">
+        <color rgba="0.023153366521000862 0.023153366521000862 0.023153366521000862 1"/>
+      </material>
+    </visual>
+    <visual>
+      <origin xyz="0.30000000000004 0.30000000000003446 -0.9065740663179903" rpy="2.1563646842988024e-14 3.504835310863548e-14 -1.5707963267948966"/>
+      <geometry>
+        <mesh filename="package://reconcycle_module_cnc/meshes/SCHUNK-5517091-finger-JGP-80-1-_-JGZ-80-12.stl"/>
+      </geometry>
+      <material name="color11">
+        <color rgba="0.023153366521000862 0.023153366521000862 0.023153366521000862 1"/>
+      </material>
+    </visual>
+    <visual>
+      <origin xyz="0.30000000000004 0.30000000000003446 -0.9065740663179903" rpy="2.1563646842988024e-14 3.504835310863548e-14 -1.5707963267948966"/>
+      <geometry>
+        <mesh filename="package://reconcycle_module_cnc/meshes/SCHUNK-9949504-limit-stop-for-MMS-P0.stl"/>
+      </geometry>
+      <material name="color2">
+        <color rgba="0.35153260827064514 0.35153260827064514 0.35153260827064514 1"/>
+      </material>
+    </visual>
+    <visual>
+      <origin xyz="0.30000000000004 0.30000000000003446 -0.9065740663179903" rpy="2.1563646842988024e-14 3.504835310863548e-14 -1.5707963267948966"/>
+      <geometry>
+        <mesh filename="package://reconcycle_module_cnc/meshes/SCHUNK-5517153-Gehaeuse-JGZ-801.stl"/>
       </geometry>
       <material name="color9">
-        <color rgba="0.5906188488006592 0.637596845626831 0.8549926280975342 1"/>
-      </material>
-    </visual>
-    <visual>
-      <origin xyz="0.30000000000004 0.30000000000003446 -0.9065740663179903" rpy="2.1563646842988024e-14 3.504835310863548e-14 -1.5707963267948966"/>
-      <geometry>
-        <mesh filename="package://reconcycle_module_cnc/meshes/PENN_ELCOM-R1290-1U_01-010-10__0.stl"/>
-      </geometry>
-      <material name="color9">
-        <color rgba="0.5906188488006592 0.637596845626831 0.8549926280975342 1"/>
-      </material>
-    </visual>
-    <visual>
-      <origin xyz="0.30000000000004 0.30000000000003446 -0.9065740663179903" rpy="2.1563646842988024e-14 3.504835310863548e-14 -1.5707963267948966"/>
-      <geometry>
-        <mesh filename="package://reconcycle_module_cnc/meshes/PENN_ELCOM-R1290-1U_R19942537480.stl"/>
-      </geometry>
-      <material name="color9">
-        <color rgba="0.5906188488006592 0.637596845626831 0.8549926280975342 1"/>
-      </material>
-    </visual>
-    <visual>
-      <origin xyz="0.30000000000004 0.30000000000003446 -0.9065740663179903" rpy="2.1563646842988024e-14 3.504835310863548e-14 -1.5707963267948966"/>
-      <geometry>
-        <mesh filename="package://reconcycle_module_cnc/meshes/PENN_ELCOM-R1290-1U_R24XX_INNER0.stl"/>
-      </geometry>
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